Commit message: add

File: ur_description/urdf/ur.xacro (robot description, xacro)
@@ -8,4 +8,5 @@
    <xacro:arg name="physical_params" default=""/>
    <xacro:arg name="visual_params" default=""/>
+   <xacro:arg name="prefix" default=""/>
    <!-- legal values:
          - hardware_interface/PositionJointInterface
@@ -19,5 +20,5 @@
    <!-- arm -->
    <xacro:ur_robot
-     prefix=""
+     prefix="$(arg prefix)"
      joint_limits_parameters_file="$(arg joint_limit_params)"
      kinematics_parameters_file="$(arg kinematics_params)"

File: ur_description/urdf/ur5e.xacro (robot description, xacro)
@@ -1,4 +1,5 @@
 <?xml version="1.0"?>
 <robot xmlns:xacro="http://wiki.ros.org/xacro" name="ur5e_robot">
+   <xacro:arg name="prefix" default=""/>
   <!--
     This is a convenience top-level xacro which loads the macro for the UR5e
@@ -15,4 +16,4 @@
   -->
   <xacro:include filename="$(find ur_description)/urdf/inc/ur5e_macro.xacro"/>
-  <xacro:ur5e_robot prefix="" />
+  <xacro:ur5e_robot prefix="$(arg prefix)" />
 </robot>

File: ur_gazebo/urdf/ur.xacro (robot description, xacro)
@@ -30,4 +30,5 @@
   <xacro:arg name="kinematics_params" default=""/>
   <xacro:arg name="visual_params" default=""/>
+  <xacro:arg name="prefix" default=""/>
   <!--
     legal values:
@@ -44,5 +45,5 @@
   <!-- Instantiate the Gazebo robot and pass it all the required arguments. -->
   <xacro:ur_robot_gazebo
-    prefix=""
+    prefix="$(arg prefix)"
     joint_limits_parameters_file="$(arg joint_limit_params)"
     kinematics_parameters_file="$(arg kinematics_params)"
@@ -64,5 +65,5 @@
   <joint name="world_joint" type="fixed">
     <parent link="world"/>
-    <child link="base_link"/>
+    <child link="$(arg prefix)base_link"/>
     <origin xyz="0 0 0" rpy="0 0 0"/>
   </joint>
